Commit message: Add ros ini file and iCubGazeboV2_5 fixed model

File: iCub/robots/iCubGazeboV2_5_fixed/model.urdf (robot description, URDF)
Before this commit: robot iCub, 189 links, 188 joints
Joints:
- joint base_fixed_joint: origin xyz=0 0 0 rpy=0 -0 0 -> xyz=0 0 1 rpy=0 -0 0

Commit message: Add world link and externalwrench plugin

File: iCub/robots/iCubGazeboV2_5_fixed/model.urdf (robot description, URDF)
Before this commit: robot iCub, 189 links, 188 joints
Links:
- added link world
Joints:
- added joint world_base_fixed_joint: type fixed, parent world, child base_link, origin xyz=0 0 0 rpy=0 -0 0, axis 0 0 0
